File: Hardware/KiCad/AmpX Open Energy Gateway/Version 2/AmpX Open Energy Gateway/AmpX Open Energy Gateway.kicad_sch (KiCad schematic)
At the start: 2 parts, among them U1 ESP32-C3-DevKitM-1

Commit message: feat: complete pcb design
Parts:
- removed U1: ESP32-C3-DevKitM-1, PCM_Espressif:ESP32-C3-DevKitM-1, symbol PCM_Espressif:ESP32-C3-DevKitM-1
- removed U2: ~, AmpX-Footprint-Library.pretty:Simple LED Module, symbol AmpX_Library_1:Simple LED Module
- added J1: POW, Connector_JST:JST_XH_B2B-XH-A_1x02_P2.50mm_Vertical, symbol Connector:Conn_01x02_Pin
- added J3: STATUS, Connector_JST:JST_XH_B5B-XH-A_1x05_P2.50mm_Vertical, symbol Connector:Conn_01x05_Pin
- added U2: W5500, Module_Ethernet_LAN_W5500_Lite.3dshapes:Module_Ethernet_LAN_W5500_Lite, symbol Module_Ethernet_LAN_W5500_Lite:Module_Ethernet_LAN_W5500_Lite
- added U3: ESP32-DEVKITC-32U, ESP32-DEVKITC-32U:MODULE_ESP32-DEVKITC-32U, symbol ESP32-DEVKITC-32U:ESP32-DEVKITC-32U
Connections:
- new net +3.3V: U2.4 (VCC), U2.5 (VCC), U3.1 (3V3)
- new net +5V: J1.1 (Pin_1), U3.19 (EXT_5V)
- new net CS: U2.11 (CS), U3.29 (IO5)
- new net DE: U3.26 (IO4)
- new net GND: J1.2 (Pin_2), U2.6 (GND), U2.7 (GND), U2.8 (GND), U3.14 (GND1), U3.32 (GND2), U3.38 (GND3)
- new net INTERNET: J3.4 (Pin_4), U3.10 (IO26)
- new net METER: J3.2 (Pin_2), U3.12 (IO14)
- new net MISO: U2.1 (MISO), U3.31 (IO19)
- new net MOSI: U2.9 (MOSI), U3.37 (IO23)
- new net POWER: J3.1 (Pin_1), U3.13 (IO12)
- new net RX: U3.27 (IO16)
- new net SCLK: U2.10 (SCK), U3.30 (IO18)
- new net SERVER: J3.5 (Pin_5), U3.9 (IO25)
- new net TX: U3.28 (IO17)
- new net WIFI: J3.3 (Pin_3), U3.11 (IO27)
- no-connect marks 17 -> 0
Other:
- company: (none) -> Ampx Europe
- title: (none) -> AmpX Open Energy Gateway
