File: Hardware/KiCad/AmpX Open Energy Gateway/Version 2/AmpX Open Energy Gateway/_autosave-AmpX Open Energy Gateway.kicad_sch (KiCad schematic)
At the start: 15 parts, among them J1 POW, J2 STATUS, J3 Status Conn Top, U2 W5500, U3 ESP32-DEVKITC-32U

Commit message: created gerbers
Connections:
- no-connect marks 26 -> 32
Changed lines of the file:
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@@
+	)
+	(no_connect
+		(at 97.79 73.66)
 	)
 	(no_connect
@@
 	)
 	(no_connect
+		(at 97.79 68.58)
+	)
+	(no_connect
 		(at 189.23 59.69)
 	)
@@
 	)
 	(no_connect
+		(at 97.79 71.12)
+	)
+	(no_connect
 		(at 184.15 137.16)
 	)
 	(no_connect
 		(at 224.79 134.62)
+	)
+	(no_connect
+		(at 97.79 63.5)
 	)
 	(no_connect
@@
 	)
 	(no_connect
+		(at 97.79 60.96)
+	)
+	(no_connect
 		(at 184.15 109.22)
 	)
 	(no_connect
+		(at 97.79 66.04)
+	)
+	(no_connect
